File: Hardware/PI-hat-PCB/WaterQualityMonitor-PI-HAT/WaterQualityMonitor-PI-HAT.kicad_sch (KiCad schematic)
At the start: 26 parts

Commit message: changed PSU voltage from 24V to 12V
Parts:
- J?: value Jack-DC 24V in -> Jack-DC 12V+
Connections:
- net 3.3V&5.5V/24V+ renamed 3.3V&5.5V/12V+
Other:
- sheet 3.3V&5.5V ports: added 12V+; removed 24V+
- sheet FluidMotors ports: added 12V+, 3.3V+; removed 24V+, 5V+
- sheet FocusMotors ports: added 12V+, 3.3V+; removed 24V+, 5V+
- sheet RaspberryPiPower ports: added 12V+; removed 24V+
Changed lines of the file:
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@@
     (effects (font (size 1.27 1.27)) (justify left bottom))
   )
-  (global_label "24V+" (shape input) (at 20.955 67.31 180) (fields_autoplaced)
+  (global_label "12V+" (shape input) (at 20.955 67.31 180) (fields_autoplaced)
     (effects (font (size 1.27 1.27)) (justify right))
-    (property "Intersheet References" "${INTERSHEET_REFS}" (id 0) (at 13.4619 67.3894 0)
+    (property "Intersheet References" "${INTERSHEET_REFS}" (id 0) (at 13.4619 67.2306 0)
       (effects (font (size 1.27 1.27)) (justify right) hide)
     )
@@
     )
   )
-  (global_label "24V+" (shape input) (at 67.31 67.31 180) (fields_autoplaced)
+  (global_label "12V+" (shape input) (at 67.31 67.31 180) (fields_autoplaced)
     (effects (font (size 1.27 1.27)) (justify right))
-    (property "Intersheet References" "${INTERSHEET_REFS}" (id 0) (at 59.8169 67.3894 0)
+    (property "Intersheet References" "${INTERSHEET_REFS}" (id 0) (at 59.8169 67.2306 0)
       (effects (font (size 1.27 1.27)) (justify right) hide)
     )
@@
     )
   )
-  (global_label "24V+" (shape input) (at 43.815 67.31 180) (fields_autoplaced)
+  (global_label "12V+" (shape input) (at 43.815 67.31 180) (fields_autoplaced)
     (effects (font (size 1.27 1.27)) (justify right))
-    (property "Intersheet References" "${INTERSHEET_REFS}" (id 0) (at 36.3219 67.3894 0)
+    (property "Intersheet References" "${INTERSHEET_REFS}" (id 0) (at 36.3219 67.2306 0)
       (effects (font (size 1.27 1.27)) (justify right) hide)
     )
@@
     (effects (font (size 1.27 1.27)) (justify right))
   )
-  (hierarchical_label "24V+" (shape input) (at 205.74 28.575 90)
+  (hierarchical_label "12V+" (shape input) (at 205.74 28.575 90)
     (effects (font (size 1.27 1.27)) (justify left))
   )
@@
   (symbol (lib_id "Connector:Jack-DC") (at 194.945 31.115 0) (unit 1)
     (in_bom yes) (on_board yes) (fields_autoplaced)
-    (property "Reference" "J?" (id 0) (at 194.945 22.479 0))
-    (property "Value" "Jack-DC 24V in" (id 1) (at 194.945 25.019 0))
+    (property "Reference" "J?" (id 0) (at 194.945 21.59 0))
+    (property "Value" "Jack-DC 12V+" (id 1) (at 194.945 24.13 0))
     (property "Footprint" "" (id 2) (at 196.215 32.131 0)
       (effects (font (size 1.27 1.27)) hide)
@@
       (effects (font (size 1.27 1.27)) (justify right))
     )
-    (pin "24V+" input (at 248.92 46.355 180)
+    (pin "12V+" input (at 248.92 46.355 180)
       (effects (font (size 1.27 1.27)) (justify left))
     )
@@
       (effects (font (size 1.27 1.27)) (justify right))
     )
-    (pin "5V+" input (at 96.52 27.94 180)
-      (effects (font (size 1.27 1.27)) (justify left))
-    )
-    (pin "24V+" input (at 96.52 25.4 180)
+    (pin "12V+" input (at 96.52 25.4 180)
       (effects (font (size 1.27 1.27)) (justify left))
     )
@@
     (pin "OB2SEC" output (at 129.54 45.72 0)
       (effects (font (size 1.27 1.27)) (justify right))
+    )
+    (pin "3.3V+" input (at 96.52 27.94 180)
+      (effects (font (size 1.27 1.27)) (justify left))
     )
   )
@@
       (effects (font (size 1.27 1.27)) (justify left top))
     )
-    (pin "24V+" input (at 248.92 33.655 180)
+    (pin "12V+" input (at 248.92 33.655 180)
       (effects (font (size 1.27 1.27)) (justify left))
     )
@@
       (effects (font (size 1.27 1.27)) (justify left top))
     )
-    (pin "24V+" input (at 142.24 25.4 180)
-      (effects (font (size 1.27 1.27)) (justify left))
-    )
-    (pin "5V+" input (at 142.24 27.94 180)
+    (pin "12V+" input (at 142.24 25.4 180)
       (effects (font (size 1.27 1.27)) (justify left))
     )
@@
     )
     (pin "STEPFOCUS" input (at 142.24 39.37 180)
+      (effects (font (size 1.27 1.27)) (justify left))
+    )
+    (pin "3.3V+" input (at 142.24 27.94 180)
       (effects (font (size 1.27 1.27)) (justify left))
     )
@@
     )
     (path "/e220ca8d-f503-491c-aac3-31543f7f0722"
-      (reference "J?") (unit 1) (value "Jack-DC 24V in") (footprint "")
+      (reference "J?") (unit 1) (value "Jack-DC 12V+") (footprint "")
     )
     (path "/2ed95514-5eec-42d9-b793-cef8be4211a9/68f34c8f-279c-4e06-8d6f-ba12c3d42e94"
