File: Hardware/PI-hat-PCB/WaterQualityMonitor-PI-HAT/FluidMotors.kicad_sch (KiCad schematic)
At the start: 2 parts

Commit message: Finished Motor drivers and started PMS again
Now I actually removed the power management system
Parts:
- U? (x2): value TMC2208_SILENTSTEPSTICK -> (none); footprint MODULE_TMC2208_SILENTSTEPSTICK -> (none)
Changed lines of the file:
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@@
     (in_bom yes) (on_board yes)
     (property "Reference" "U?" (id 0) (at 177.8 78.74 0))
-    (property "Value" "TMC2208_SILENTSTEPSTICK" (id 1) (at 177.8 81.28 0))
-    (property "Footprint" "MODULE_TMC2208_SILENTSTEPSTICK" (id 2) (at 162.56 123.19 0)
+    (property "Value" "" (id 1) (at 177.8 81.28 0))
+    (property "Footprint" "" (id 2) (at 162.56 123.19 0)
       (effects (font (size 1.27 1.27)) (justify left bottom) hide)
     )
@@
       (effects (font (size 1.27 1.27)) hide)
     )
-    (property "Value" "GND" (id 1) (at 196.85 123.19 0))
+    (property "Value" "" (id 1) (at 196.85 123.19 0))
     (property "Footprint" "" (id 2) (at 196.85 118.11 0)
       (effects (font (size 1.27 1.27)) hide)
@@
       (effects (font (size 1.27 1.27)) hide)
     )
-    (property "Value" "GND" (id 1) (at 157.48 96.52 0))
+    (property "Value" "" (id 1) (at 157.48 96.52 0))
     (property "Footprint" "" (id 2) (at 157.48 91.44 0)
       (effects (font (size 1.27 1.27)) hide)
@@
       (effects (font (size 1.27 1.27)) hide)
     )
-    (property "Value" "GND" (id 1) (at 135.89 123.19 0))
+    (property "Value" "" (id 1) (at 135.89 123.19 0))
     (property "Footprint" "" (id 2) (at 135.89 118.11 0)
       (effects (font (size 1.27 1.27)) hide)
@@
       (effects (font (size 1.27 1.27)) hide)
     )
-    (property "Value" "GND" (id 1) (at 96.52 96.52 0))
+    (property "Value" "" (id 1) (at 96.52 96.52 0))
     (property "Footprint" "" (id 2) (at 96.52 91.44 0)
       (effects (font (size 1.27 1.27)) hide)
@@
     (in_bom yes) (on_board yes) (fields_autoplaced)
     (property "Reference" "U?" (id 0) (at 116.84 78.74 0))
-    (property "Value" "TMC2208_SILENTSTEPSTICK" (id 1) (at 116.84 81.28 0))
-    (property "Footprint" "MODULE_TMC2208_SILENTSTEPSTICK" (id 2) (at 101.6 123.19 0)
+    (property "Value" "" (id 1) (at 116.84 81.28 0))
+    (property "Footprint" "" (id 2) (at 101.6 123.19 0)
       (effects (font (size 1.27 1.27)) (justify left bottom) hide)
     )

Commit message: Finished powermanagementsystem
added RPI powersupply
added 5V and 3.3V power supply
changed some components (errors)
Parts:
- U? (x2): value (none) -> TMC2208_SILENTSTEPSTICK; footprint (none) -> MODULE_TMC2208_SILENTSTEPSTICK
Changed lines of the file:
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@@
     (in_bom yes) (on_board yes)
     (property "Reference" "U?" (id 0) (at 177.8 78.74 0))
-    (property "Value" "" (id 1) (at 177.8 81.28 0))
-    (property "Footprint" "" (id 2) (at 162.56 123.19 0)
+    (property "Value" "TMC2208_SILENTSTEPSTICK" (id 1) (at 177.8 81.28 0))
+    (property "Footprint" "MODULE_TMC2208_SILENTSTEPSTICK" (id 2) (at 162.56 123.19 0)
       (effects (font (size 1.27 1.27)) (justify left bottom) hide)
     )
@@
       (effects (font (size 1.27 1.27)) hide)
     )
-    (property "Value" "" (id 1) (at 196.85 123.19 0))
+    (property "Value" "GND" (id 1) (at 196.85 123.19 0))
     (property "Footprint" "" (id 2) (at 196.85 118.11 0)
       (effects (font (size 1.27 1.27)) hide)
@@
       (effects (font (size 1.27 1.27)) hide)
     )
-    (property "Value" "" (id 1) (at 157.48 96.52 0))
+    (property "Value" "GND" (id 1) (at 157.48 96.52 0))
     (property "Footprint" "" (id 2) (at 157.48 91.44 0)
       (effects (font (size 1.27 1.27)) hide)
@@
       (effects (font (size 1.27 1.27)) hide)
     )
-    (property "Value" "" (id 1) (at 135.89 123.19 0))
+    (property "Value" "GND" (id 1) (at 135.89 123.19 0))
     (property "Footprint" "" (id 2) (at 135.89 118.11 0)
       (effects (font (size 1.27 1.27)) hide)
@@
       (effects (font (size 1.27 1.27)) hide)
     )
-    (property "Value" "" (id 1) (at 96.52 96.52 0))
+    (property "Value" "GND" (id 1) (at 96.52 96.52 0))
     (property "Footprint" "" (id 2) (at 96.52 91.44 0)
       (effects (font (size 1.27 1.27)) hide)
@@
     (in_bom yes) (on_board yes) (fields_autoplaced)
     (property "Reference" "U?" (id 0) (at 116.84 78.74 0))
-    (property "Value" "" (id 1) (at 116.84 81.28 0))
-    (property "Footprint" "" (id 2) (at 101.6 123.19 0)
+    (property "Value" "TMC2208_SILENTSTEPSTICK" (id 1) (at 116.84 81.28 0))
+    (property "Footprint" "MODULE_TMC2208_SILENTSTEPSTICK" (id 2) (at 101.6 123.19 0)
       (effects (font (size 1.27 1.27)) (justify left bottom) hide)
     )

Commit message: Enhanced schematics
Moved protection circuits to main schematic
changed tmc2208 VIO to 3.3V (5V is also fine)
added fuses to heat and cooling schematic
Connections:
- net 5V+ renamed 3.3V+
Changed lines of the file:
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@@
     (effects (font (size 1.27 1.27)) (justify left))
   )
-  (hierarchical_label "5V+" (shape input) (at 134.62 88.9 0)
+  (hierarchical_label "3.3V+" (shape input) (at 134.62 88.9 0)
     (effects (font (size 1.27 1.27)) (justify left))
   )
@@
   (hierarchical_label "DIRSEC" (shape input) (at 160.02 99.06 180)
     (effects (font (size 1.27 1.27)) (justify right))
-  )
-  (hierarchical_label "5V+" (shape input) (at 195.58 88.9 0)
-    (effects (font (size 1.27 1.27)) (justify left))
   )
   (hierarchical_label "VREF" (shape input) (at 134.62 95.25 0)
@@
     (effects (font (size 1.27 1.27)) (justify left))
   )
+  (hierarchical_label "3.3V+" (shape input) (at 195.58 88.9 0)
+    (effects (font (size 1.27 1.27)) (justify left))
+  )

Commit message: changed PSU voltage from 24V to 12V
Connections:
- net 24V+ renamed 12V+
Changed lines of the file:
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@@
     (effects (font (size 1.27 1.27)) (justify left))
   )
-  (hierarchical_label "24V+" (shape input) (at 134.62 91.44 0)
+  (hierarchical_label "12V+" (shape input) (at 134.62 91.44 0)
     (effects (font (size 1.27 1.27)) (justify left))
   )
@@
     (effects (font (size 1.27 1.27)) (justify left))
   )
-  (hierarchical_label "24V+" (shape input) (at 195.58 91.44 0)
+  (hierarchical_label "12V+" (shape input) (at 195.58 91.44 0)
     (effects (font (size 1.27 1.27)) (justify left))
   )

Commit message: assigent footprints to all current components
I chose 1206smd handsolderable for caps and resistors and inductors, may need to be revised
Parts:
- U3, U4: renamed from U?; footprint MODULE_TMC2208_SILENTSTEPSTICK -> Footprints:TMC2208_SILENTSTEPSTICK
Changed lines of the file:
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@@
   (symbol (lib_name "TMC2208_SILENTSTEPSTICK_1") (lib_id "TMC2208_SILENTSTEPSTICK:TMC2208_SILENTSTEPSTICK") (at 177.8 104.14 0) (unit 1)
     (in_bom yes) (on_board yes)
-    (property "Reference" "U?" (id 0) (at 177.8 78.74 0))
+    (property "Reference" "U4" (id 0) (at 177.8 78.74 0))
     (property "Value" "TMC2208_SILENTSTEPSTICK" (id 1) (at 177.8 81.28 0))
-    (property "Footprint" "MODULE_TMC2208_SILENTSTEPSTICK" (id 2) (at 162.56 123.19 0)
+    (property "Footprint" "Footprints:TMC2208_SILENTSTEPSTICK" (id 2) (at 162.56 123.19 0)
       (effects (font (size 1.27 1.27)) (justify left bottom) hide)
     )
@@
   (symbol (lib_name "TMC2208_SILENTSTEPSTICK_1") (lib_id "TMC2208_SILENTSTEPSTICK:TMC2208_SILENTSTEPSTICK") (at 116.84 104.14 0) (unit 1)
     (in_bom yes) (on_board yes) (fields_autoplaced)
-    (property "Reference" "U?" (id 0) (at 116.84 78.74 0))
+    (property "Reference" "U3" (id 0) (at 116.84 78.74 0))
     (property "Value" "TMC2208_SILENTSTEPSTICK" (id 1) (at 116.84 81.28 0))
-    (property "Footprint" "MODULE_TMC2208_SILENTSTEPSTICK" (id 2) (at 101.6 123.19 0)
+    (property "Footprint" "Footprints:TMC2208_SILENTSTEPSTICK" (id 2) (at 101.6 123.19 0)
       (effects (font (size 1.27 1.27)) (justify left bottom) hide)
     )
