File: Hardware/PI-hat-PCB/WaterQualityMonitor-PI-HAT/FluidMotors.kicad_sch (KiCad schematic)
At the start: 2 parts, among them U3 TMC2208_SILENTSTEPSTICK, U4 TMC2208_SILENTSTEPSTICK

Commit message: added resistors to ms1 and ms2 of tmc2208 for micro stepping
Parts:
- added R? (x4): 22k, symbol Device:R
Connections:
- net 3.3V+: now also R?.2, R?.2, R?.2, R?.2
- net at U4.JP1_6 (MS2): now also R?.1
- net at U4.JP1_7 (MS1): now also R?.1
- net at U3.JP1_6 (MS2): now also R?.1
- net at U3.JP1_7 (MS1): now also R?.1
- no-connect marks 10 -> 6
Other:
- moved on the sheet: U4

Commit message: added left over gpio connector
Parts:
- R20, R21, R22, R23: renamed from R?; footprint (none) -> Resistor_SMD:R_1206_3216Metric_Pad1.30x1.75mm_HandSolder
Changed lines of the file:
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@@
   (symbol (lib_id "Device:R") (at 153.67 114.3 0) (unit 1)
     (in_bom yes) (on_board yes)
-    (property "Reference" "R?" (id 0) (at 156.21 113.0299 0)
+    (property "Reference" "R22" (id 0) (at 156.21 113.0299 0)
       (effects (font (size 1.27 1.27)) (justify left))
     )
@@
       (effects (font (size 1.27 1.27)) (justify left))
     )
-    (property "Footprint" "" (id 2) (at 151.892 114.3 90)
+    (property "Footprint" "Resistor_SMD:R_1206_3216Metric_Pad1.30x1.75mm_HandSolder" (id 2) (at 151.892 114.3 90)
       (effects (font (size 1.27 1.27)) hide)
     )
@@
   (symbol (lib_id "Device:R") (at 92.075 114.3 0) (unit 1)
     (in_bom yes) (on_board yes)
-    (property "Reference" "R?" (id 0) (at 94.615 113.0299 0)
+    (property "Reference" "R21" (id 0) (at 94.615 113.0299 0)
       (effects (font (size 1.27 1.27)) (justify left))
     )
@@
       (effects (font (size 1.27 1.27)) (justify left))
     )
-    (property "Footprint" "" (id 2) (at 90.297 114.3 90)
+    (property "Footprint" "Resistor_SMD:R_1206_3216Metric_Pad1.30x1.75mm_HandSolder" (id 2) (at 90.297 114.3 90)
       (effects (font (size 1.27 1.27)) hide)
     )
@@
   (symbol (lib_id "Device:R") (at 160.02 114.3 0) (unit 1)
     (in_bom yes) (on_board yes)
-    (property "Reference" "R?" (id 0) (at 162.56 113.0299 0)
+    (property "Reference" "R23" (id 0) (at 162.56 113.0299 0)
       (effects (font (size 1.27 1.27)) (justify left))
     )
@@
       (effects (font (size 1.27 1.27)) (justify left))
     )
-    (property "Footprint" "" (id 2) (at 158.242 114.3 90)
+    (property "Footprint" "Resistor_SMD:R_1206_3216Metric_Pad1.30x1.75mm_HandSolder" (id 2) (at 158.242 114.3 90)
       (effects (font (size 1.27 1.27)) hide)
     )
@@
   (symbol (lib_id "Device:R") (at 85.725 114.3 0) (unit 1)
     (in_bom yes) (on_board yes)
-    (property "Reference" "R?" (id 0) (at 88.265 113.0299 0)
+    (property "Reference" "R20" (id 0) (at 88.265 113.0299 0)
       (effects (font (size 1.27 1.27)) (justify left))
     )
@@
       (effects (font (size 1.27 1.27)) (justify left))
     )
-    (property "Footprint" "" (id 2) (at 83.947 114.3 90)
+    (property "Footprint" "Resistor_SMD:R_1206_3216Metric_Pad1.30x1.75mm_HandSolder" (id 2) (at 83.947 114.3 90)
       (effects (font (size 1.27 1.27)) hide)
     )

Commit message: added some test points
Parts:
- added TP? (x2): TestPoint, symbol Connector:TestPoint
Connections:
- net STEPMAIN: now also TP?.1
- net STEPSEC: now also TP?.1
Changed lines of the file:
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@@
     (effects (font (size 1.27 1.27)) (justify left))
+  )
+  (symbol (lib_id "Connector:TestPoint") (at 166.37 101.6 180) (unit 1)
+    (in_bom yes) (on_board yes)
+    (property "Reference" "TP?" (id 0) (at 163.83 104.14 0))
+    (property "Value" "TestPoint" (id 1) (at 166.37 106.68 0)
+      (effects (font (size 1.27 1.27)) hide)
+    )
+    (property "Footprint" "" (id 2) (at 161.29 101.6 0)
+      (effects (font (size 1.27 1.27)) hide)
+    )
+    (property "Datasheet" "~" (id 3) (at 161.29 101.6 0)
+      (effects (font (size 1.27 1.27)) hide)
+    )
+    (pin "1")
   )
   (symbol (lib_name "TMC2208_SILENTSTEPSTICK_1") (lib_id "TMC2208_SILENTSTEPSTICK:TMC2208_SILENTSTEPSTICK") (at 184.15 104.14 0) (unit 1)
@@
     (pin "2")
   )
+  (symbol (lib_id "Connector:TestPoint") (at 99.06 101.6 180) (unit 1)
+    (in_bom yes) (on_board yes)
+    (property "Reference" "TP?" (id 0) (at 96.52 104.14 0))
+    (property "Value" "TestPoint" (id 1) (at 99.06 106.68 0)
+      (effects (font (size 1.27 1.27)) hide)
+    )
+    (property "Footprint" "" (id 2) (at 93.98 101.6 0)
+      (effects (font (size 1.27 1.27)) hide)
+    )
+    (property "Datasheet" "~" (id 3) (at 93.98 101.6 0)
+      (effects (font (size 1.27 1.27)) hide)
+    )
+    (pin "1")
+  )
 )

Commit message: created new bom and experimented with BOM file
Parts:
- TP3, TP4: renamed from TP?; footprint (none) -> TestPoint:TestPoint_Keystone_5019_Minature
Changed lines of the file:
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@@
   (symbol (lib_id "Connector:TestPoint") (at 166.37 101.6 180) (unit 1)
     (in_bom yes) (on_board yes)
-    (property "Reference" "TP?" (id 0) (at 163.83 104.14 0))
+    (property "Reference" "TP4" (id 0) (at 163.83 104.14 0))
     (property "Value" "TestPoint" (id 1) (at 166.37 106.68 0)
       (effects (font (size 1.27 1.27)) hide)
     )
-    (property "Footprint" "" (id 2) (at 161.29 101.6 0)
+    (property "Footprint" "TestPoint:TestPoint_Keystone_5019_Minature" (id 2) (at 161.29 101.6 0)
       (effects (font (size 1.27 1.27)) hide)
     )
@@
   (symbol (lib_id "Connector:TestPoint") (at 99.06 101.6 180) (unit 1)
     (in_bom yes) (on_board yes)
-    (property "Reference" "TP?" (id 0) (at 96.52 104.14 0))
+    (property "Reference" "TP3" (id 0) (at 96.52 104.14 0))
     (property "Value" "TestPoint" (id 1) (at 99.06 106.68 0)
       (effects (font (size 1.27 1.27)) hide)
     )
-    (property "Footprint" "" (id 2) (at 93.98 101.6 0)
-      (effects (font (size 1.27 1.27)) hide)
-    )
+    (property "Footprint" "TestPoint:TestPoint_Keystone_5019_Minature" (id 2) (at 93.98 101.6 0)
+      (effects (font (size 1.27 1.27)) hide)
+    )

Commit message: changed testpoint footprints
Parts:
- TP3, TP4: footprint TestPoint:TestPoint_Keystone_5019_Minature -> TestPoint:TestPoint_Bridge_Pitch7.62mm_Drill1.3mm
Changed lines of the file:
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@@
       (effects (font (size 1.27 1.27)) hide)
     )
-    (property "Footprint" "TestPoint:TestPoint_Keystone_5019_Minature" (id 2) (at 161.29 101.6 0)
+    (property "Footprint" "TestPoint:TestPoint_Bridge_Pitch7.62mm_Drill1.3mm" (id 2) (at 161.29 101.6 0)
       (effects (font (size 1.27 1.27)) hide)
     )
@@
       (effects (font (size 1.27 1.27)) hide)
     )
-    (property "Footprint" "TestPoint:TestPoint_Keystone_5019_Minature" (id 2) (at 93.98 101.6 0)
-      (effects (font (size 1.27 1.27)) hide)
-    )
+    (property "Footprint" "TestPoint:TestPoint_Bridge_Pitch7.62mm_Drill1.3mm" (id 2) (at 93.98 101.6 0)
+      (effects (font (size 1.27 1.27)) hide)
+    )

Commit message: changed name from primary (main) to PRI (logical)
Connections:
- net GND: no longer U3.JP1_8 (EN), U4.JP1_8 (EN)
- net DIAGMAIN renamed DIAGPRI
- net DIRMAIN renamed DIRPRI
- net OA1MAIN renamed OA1PRI
- net OA2MAIN renamed OA2PRI
- net OB1MAIN renamed OB1PRI
- net OB2MAIN renamed OB2PRI
- net STEPMAIN renamed STEPPRI
- new net ENPRI: U3.JP1_8 (EN)
- new net ENSEC: U4.JP1_8 (EN)
Changed lines of the file:
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@@
-    (stroke (width 0) (type default) (color 0 0 0 0))
-  )
-  (wire (pts (xy 163.83 90.17) (xy 163.83 91.44))
     (stroke (width 0) (type default) (color 0 0 0 0))
   )
@@
     (stroke (width 0) (type default) (color 0 0 0 0))
   )
-  (wire (pts (xy 166.37 90.17) (xy 163.83 90.17))
-    (stroke (width 0) (type default) (color 0 0 0 0))
-  )
   (wire (pts (xy 85.725 106.68) (xy 85.725 110.49))
     (stroke (width 0) (type default) (color 0 0 0 0))
@@
     (stroke (width 0) (type default) (color 0 0 0 0))
   )
-  (wire (pts (xy 96.52 90.17) (xy 96.52 91.44))
-    (stroke (width 0) (type default) (color 0 0 0 0))
-  )
-  (wire (pts (xy 99.06 90.17) (xy 96.52 90.17))
-    (stroke (width 0) (type default) (color 0 0 0 0))
-  )
   (wire (pts (xy 203.2 118.11) (xy 203.2 116.84))
     (stroke (width 0) (type default) (color 0 0 0 0))
@@
     (effects (font (size 1.27 1.27)) (justify left))
   )
-  (hierarchical_label "DIAGMAIN" (shape output) (at 134.62 113.03 0)
+  (hierarchical_label "DIAGPRI" (shape output) (at 134.62 113.03 0)
     (effects (font (size 1.27 1.27)) (justify left))
   )
@@
     (effects (font (size 1.27 1.27)) (justify left))
   )
-  (hierarchical_label "STEPMAIN" (shape input) (at 99.06 101.6 180)
+  (hierarchical_label "STEPPRI" (shape input) (at 99.06 101.6 180)
     (effects (font (size 1.27 1.27)) (justify right))
   )
@@
     (effects (font (size 1.27 1.27)) (justify left))
   )
-  (hierarchical_label "OA2MAIN" (shape output) (at 134.62 101.6 0)
+  (hierarchical_label "OA2PRI" (shape output) (at 134.62 101.6 0)
     (effects (font (size 1.27 1.27)) (justify left))
   )
@@
     (effects (font (size 1.27 1.27)) (justify left))
   )
+  (hierarchical_label "ENSEC" (shape input) (at 166.37 90.17 180)
+    (effects (font (size 1.27 1.27)) (justify right))
+  )
+  (hierarchical_label "ENPRI" (shape input) (at 99.06 90.17 180)
+    (effects (font (size 1.27 1.27)) (justify right))
+  )
   (hierarchical_label "STEPSEC" (shape input) (at 166.37 101.6 180)
     (effects (font (size 1.27 1.27)) (justify right))
@@
     (effects (font (size 1.27 1.27)) (justify left))
   )
-  (hierarchical_label "OA1MAIN" (shape output) (at 134.62 99.06 0)
+  (hierarchical_label "OA1PRI" (shape output) (at 134.62 99.06 0)
     (effects (font (size 1.27 1.27)) (justify left))
   )
@@
     (effects (font (size 1.27 1.27)) (justify left))
   )
-  (hierarchical_label "OB2MAIN" (shape output) (at 134.62 106.68 0)
-    (effects (font (size 1.27 1.27)) (justify left))
-  )
-  (hierarchical_label "OB1MAIN" (shape output) (at 134.62 104.14 0)
-    (effects (font (size 1.27 1.27)) (justify left))
-  )
-  (hierarchical_label "DIRMAIN" (shape input) (at 99.06 99.06 180)
+  (hierarchical_label "OB2PRI" (shape output) (at 134.62 106.68 0)
+    (effects (font (size 1.27 1.27)) (justify left))
+  )
+  (hierarchical_label "OB1PRI" (shape output) (at 134.62 104.14 0)
+    (effects (font (size 1.27 1.27)) (justify left))
+  )
+  (hierarchical_label "DIRPRI" (shape input) (at 99.06 99.06 180)
     (effects (font (size 1.27 1.27)) (justify right))
   )
@@
     (pin "2")
   )
-  (symbol (lib_id "power:GND") (at 163.83 91.44 0) (unit 1)
-    (in_bom yes) (on_board yes) (fields_autoplaced)
-    (property "Reference" "#PWR0111" (id 0) (at 163.83 97.79 0)
-      (effects (font (size 1.27 1.27)) hide)
-    )
-    (property "Value" "GND" (id 1) (at 163.83 96.52 0))
-    (property "Footprint" "" (id 2) (at 163.83 91.44 0)
-      (effects (font (size 1.27 1.27)) hide)
-    )
-    (property "Datasheet" "" (id 3) (at 163.83 91.44 0)
-      (effects (font (size 1.27 1.27)) hide)
-    )
-    (pin "1")
-  )
   (symbol (lib_id "power:GND") (at 135.89 118.11 0) (unit 1)
     (in_bom yes) (on_board yes) (fields_autoplaced)
@@
       (effects (font (size 1.27 1.27)) hide)
     )
-    (pin "1")
-  )
-  (symbol (lib_id "power:GND") (at 96.52 91.44 0) (unit 1)
-    (in_bom yes) (on_board yes) (fields_autoplaced)
-    (property "Reference" "#PWR0112" (id 0) (at 96.52 97.79 0)
-      (effects (font (size 1.27 1.27)) hide)
-    )
-    (property "Value" "GND" (id 1) (at 96.52 96.52 0))
-    (property "Footprint" "" (id 2) (at 96.52 91.44 0)
-      (effects (font (size 1.27 1.27)) hide)
-    )
-    (property "Datasheet" "" (id 3) (at 96.52 91.44 0)
-      (effects (font (size 1.27 1.27)) hide)
-    )

Commit message: enh schematic
added power pins breakout
replaced common ground with specific ground labels
Connections:
- net GND renamed GNDPWR
Changed lines of the file:
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@@
     (pin "VREF")
-  )
-  (symbol (lib_id "power:GND") (at 203.2 118.11 0) (unit 1)
-    (in_bom yes) (on_board yes) (fields_autoplaced)
-    (property "Reference" "#PWR0114" (id 0) (at 203.2 124.46 0)
-      (effects (font (size 1.27 1.27)) hide)
-    )
-    (property "Value" "GND" (id 1) (at 203.2 123.19 0))
-    (property "Footprint" "" (id 2) (at 203.2 118.11 0)
-      (effects (font (size 1.27 1.27)) hide)
-    )
-    (property "Datasheet" "" (id 3) (at 203.2 118.11 0)
-      (effects (font (size 1.27 1.27)) hide)
-    )
-    (pin "1")
   )
   (symbol (lib_id "Device:R") (at 153.67 114.3 0) (unit 1)
@@
     (pin "2")
   )
-  (symbol (lib_id "power:GND") (at 135.89 118.11 0) (unit 1)
+  (symbol (lib_id "power:GNDPWR") (at 203.2 118.11 0) (unit 1)
     (in_bom yes) (on_board yes) (fields_autoplaced)
-    (property "Reference" "#PWR0113" (id 0) (at 135.89 124.46 0)
+    (property "Reference" "#PWR017" (id 0) (at 203.2 123.19 0)
       (effects (font (size 1.27 1.27)) hide)
     )
-    (property "Value" "GND" (id 1) (at 135.89 123.19 0))
-    (property "Footprint" "" (id 2) (at 135.89 118.11 0)
+    (property "Value" "GNDPWR" (id 1) (at 203.073 122.555 0))
+    (property "Footprint" "" (id 2) (at 203.2 119.38 0)
       (effects (font (size 1.27 1.27)) hide)
     )
-    (property "Datasheet" "" (id 3) (at 135.89 118.11 0)
+    (property "Datasheet" "" (id 3) (at 203.2 119.38 0)
       (effects (font (size 1.27 1.27)) hide)
     )
+    (pin "1")
+  )
+  (symbol (lib_id "power:GNDPWR") (at 135.89 118.11 0) (unit 1)
+    (in_bom yes) (on_board yes) (fields_autoplaced)
+    (property "Reference" "#PWR016" (id 0) (at 135.89 123.19 0)
+      (effects (font (size 1.27 1.27)) hide)
+    )
+    (property "Value" "GNDPWR" (id 1) (at 135.763 122.555 0))
+    (property "Footprint" "" (id 2) (at 135.89 119.38 0)
+      (effects (font (size 1.27 1.27)) hide)
+    )
+    (property "Datasheet" "" (id 3) (at 135.89 119.38 0)
+      (effects (font (size 1.27 1.27)) hide)
+    )

Commit message: finished up V1.0. Review required
Other:
- company: (none) -> HAN
- title: (none) -> Water Quality Monitor
Changed lines of the file:
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@@
 (kicad_sch (version 20211123) (generator eeschema)
   (paper "A4")
+  (title_block
+    (title "Water Quality Monitor")
+    (rev "1")
+    (company "HAN")
+    (comment 1 "Casper R. Tak")
+  )
   (junction (at 157.48 118.11) (diameter 0) (color 0 0 0 0)
   )
