File: Hardware/PI-hat-PCB/WaterQualityMonitor-PI-HAT/FocusMotors.kicad_sch (KiCad schematic)
At the start: 4 parts, among them U6 TMC2208_SILENTSTEPSTICK, U7 DRV8838

Commit message: added resistors to ms1 and ms2 of tmc2208 for micro stepping
Parts:
- added R? (x2): 22k, symbol Device:R
Connections:
- net 3.3V+: now also R?.2, R?.2
- net at U6.JP1_6 (MS2): now also R?.1
- net at U6.JP1_7 (MS1): now also R?.1
- no-connect marks 5 -> 3
Changed lines of the file:
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@@
   (junction (at 177.8 111.125) (diameter 0) (color 0 0 0 0)
+  )
+  (junction (at 97.155 114.3) (diameter 0) (color 0 0 0 0)
   )
   (junction (at 177.8 98.425) (diameter 0) (color 0 0 0 0)
@@
   (no_connect (at 106.045 110.49))
   (no_connect (at 106.045 113.03))
-  (no_connect (at 106.045 102.87))
-  (no_connect (at 106.045 105.41))
   (wire (pts (xy 192.405 98.425) (xy 192.405 88.265))
     (stroke (width 0) (type default) (color 0 0 0 0))
@@
     (stroke (width 0) (type default) (color 0 0 0 0))
   )
+  (wire (pts (xy 106.045 102.87) (xy 93.345 102.87))
+    (stroke (width 0) (type default) (color 0 0 0 0))
+  )
   (wire (pts (xy 186.055 122.555) (xy 185.42 122.555))
     (stroke (width 0) (type default) (color 0 0 0 0))
@@
     (stroke (width 0) (type default) (color 0 0 0 0))
   )
+  (wire (pts (xy 93.345 114.3) (xy 97.155 114.3))
+    (stroke (width 0) (type default) (color 0 0 0 0))
+  )
   (wire (pts (xy 106.045 86.36) (xy 103.505 86.36))
     (stroke (width 0) (type default) (color 0 0 0 0))
@@
     (stroke (width 0) (type default) (color 0 0 0 0))
   )
+  (wire (pts (xy 106.045 105.41) (xy 99.695 105.41))
+    (stroke (width 0) (type default) (color 0 0 0 0))
+  )
   (wire (pts (xy 103.505 86.36) (xy 103.505 87.63))
     (stroke (width 0) (type default) (color 0 0 0 0))
   )
+  (wire (pts (xy 97.155 114.3) (xy 99.695 114.3))
+    (stroke (width 0) (type default) (color 0 0 0 0))
+  )
   (wire (pts (xy 177.8 98.425) (xy 177.8 111.125))
     (stroke (width 0) (type default) (color 0 0 0 0))
   )
+  (wire (pts (xy 99.695 105.41) (xy 99.695 106.68))
+    (stroke (width 0) (type default) (color 0 0 0 0))
+  )
   (wire (pts (xy 186.055 97.155) (xy 186.055 122.555))
     (stroke (width 0) (type default) (color 0 0 0 0))
   )
+  (wire (pts (xy 93.345 102.87) (xy 93.345 106.68))
+    (stroke (width 0) (type default) (color 0 0 0 0))
+  )
   (wire (pts (xy 180.34 98.425) (xy 180.975 98.425))
     (stroke (width 0) (type default) (color 0 0 0 0))
@@
     (stroke (width 0) (type default) (color 0 0 0 0))
   )
+  (wire (pts (xy 97.155 114.3) (xy 97.155 118.11))
+    (stroke (width 0) (type default) (color 0 0 0 0))
+  )
   (hierarchical_label "VREF" (shape input) (at 141.605 91.44 0)
     (effects (font (size 1.27 1.27)) (justify left))
   )
   (hierarchical_label "OA2FOCUS" (shape output) (at 141.605 97.79 0)
+    (effects (font (size 1.27 1.27)) (justify left))
+  )
+  (hierarchical_label "3.3V+" (shape input) (at 97.155 118.11 0)
     (effects (font (size 1.27 1.27)) (justify left))
   )
@@
     (pin "2")
   )
+  (symbol (lib_id "Device:R") (at 93.345 110.49 0) (unit 1)
+    (in_bom yes) (on_board yes)
+    (property "Reference" "R?" (id 0) (at 95.885 109.2199 0)
+      (effects (font (size 1.27 1.27)) (justify left))
+    )
+    (property "Value" "22k" (id 1) (at 94.615 111.76 0)
+      (effects (font (size 1.27 1.27)) (justify left))
+    )
+    (property "Footprint" "" (id 2) (at 91.567 110.49 90)
+      (effects (font (size 1.27 1.27)) hide)
+    )
+    (property "Datasheet" "~" (id 3) (at 93.345 110.49 0)
+      (effects (font (size 1.27 1.27)) hide)
+    )
+    (pin "1")
+    (pin "2")
+  )
   (symbol (lib_id "power:GND") (at 142.875 114.3 0) (unit 1)
     (in_bom yes) (on_board yes) (fields_autoplaced)
@@
     (pin "1")
   )
+  (symbol (lib_id "Device:R") (at 99.695 110.49 0) (unit 1)
+    (in_bom yes) (on_board yes)
+    (property "Reference" "R?" (id 0) (at 102.235 109.2199 0)
+      (effects (font (size 1.27 1.27)) (justify left))
+    )
+    (property "Value" "22k" (id 1) (at 100.965 111.76 0)
+      (effects (font (size 1.27 1.27)) (justify left))
+    )
+    (property "Footprint" "" (id 2) (at 97.917 110.49 90)
+      (effects (font (size 1.27 1.27)) hide)
+    )
+    (property "Datasheet" "~" (id 3) (at 99.695 110.49 0)
+      (effects (font (size 1.27 1.27)) hide)
+    )
+    (pin "1")
+    (pin "2")
+  )
 )

Commit message: added left over gpio connector
Parts:
- R24, R25: renamed from R?; footprint (none) -> Resistor_SMD:R_1206_3216Metric_Pad1.30x1.75mm_HandSolder
Changed lines of the file:
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@@
   (symbol (lib_id "Device:R") (at 93.345 110.49 0) (unit 1)
     (in_bom yes) (on_board yes)
-    (property "Reference" "R?" (id 0) (at 95.885 109.2199 0)
+    (property "Reference" "R24" (id 0) (at 95.885 109.2199 0)
       (effects (font (size 1.27 1.27)) (justify left))
     )
@@
       (effects (font (size 1.27 1.27)) (justify left))
     )
-    (property "Footprint" "" (id 2) (at 91.567 110.49 90)
+    (property "Footprint" "Resistor_SMD:R_1206_3216Metric_Pad1.30x1.75mm_HandSolder" (id 2) (at 91.567 110.49 90)
       (effects (font (size 1.27 1.27)) hide)
     )
@@
   (symbol (lib_id "Device:R") (at 99.695 110.49 0) (unit 1)
     (in_bom yes) (on_board yes)
-    (property "Reference" "R?" (id 0) (at 102.235 109.2199 0)
+    (property "Reference" "R25" (id 0) (at 102.235 109.2199 0)
       (effects (font (size 1.27 1.27)) (justify left))
     )
@@
       (effects (font (size 1.27 1.27)) (justify left))
     )
-    (property "Footprint" "" (id 2) (at 97.917 110.49 90)
+    (property "Footprint" "Resistor_SMD:R_1206_3216Metric_Pad1.30x1.75mm_HandSolder" (id 2) (at 97.917 110.49 90)
       (effects (font (size 1.27 1.27)) hide)
     )

Commit message: enh schematic
added power pins breakout
replaced common ground with specific ground labels
Connections:
- net GND: no longer C14.1, C15.1, U6.JP2_2 (GND), U6.JP2_8 (GND), U7.4 (GND), U7.9 (GND)
- new net GNDPWR: C14.1, C15.1, U6.JP2_2 (GND), U6.JP2_8 (GND), U7.4 (GND), U7.9 (GND)
Changed lines of the file:
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@@
     (effects (font (size 1.27 1.27)) (justify right))
+  )
+  (symbol (lib_id "power:GNDPWR") (at 142.875 114.3 0) (unit 1)
+    (in_bom yes) (on_board yes) (fields_autoplaced)
+    (property "Reference" "#PWR023" (id 0) (at 142.875 119.38 0)
+      (effects (font (size 1.27 1.27)) hide)
+    )
+    (property "Value" "GNDPWR" (id 1) (at 142.748 118.745 0))
+    (property "Footprint" "" (id 2) (at 142.875 115.57 0)
+      (effects (font (size 1.27 1.27)) hide)
+    )
+    (property "Datasheet" "" (id 3) (at 142.875 115.57 0)
+      (effects (font (size 1.27 1.27)) hide)
+    )
+    (pin "1")
   )
   (symbol (lib_name "TMC2208_SILENTSTEPSTICK_1") (lib_id "TMC2208_SILENTSTEPSTICK:TMC2208_SILENTSTEPSTICK") (at 123.825 100.33 0) (unit 1)
@@
     (pin "VREF")
   )
+  (symbol (lib_id "power:GNDPWR") (at 174.625 99.06 0) (unit 1)
+    (in_bom yes) (on_board yes) (fields_autoplaced)
+    (property "Reference" "#PWR024" (id 0) (at 174.625 104.14 0)
+      (effects (font (size 1.27 1.27)) hide)
+    )
+    (property "Value" "GNDPWR" (id 1) (at 174.498 103.505 0))
+    (property "Footprint" "" (id 2) (at 174.625 100.33 0)
+      (effects (font (size 1.27 1.27)) hide)
+    )
+    (property "Datasheet" "" (id 3) (at 174.625 100.33 0)
+      (effects (font (size 1.27 1.27)) hide)
+    )
+    (pin "1")
+  )
   (symbol (lib_id "Device:C") (at 181.61 122.555 90) (unit 1)
     (in_bom yes) (on_board yes)
@@
     )
     (property "Datasheet" "" (id 3) (at 103.505 87.63 0)
-      (effects (font (size 1.27 1.27)) hide)
-    )
-    (pin "1")
-  )
-  (symbol (lib_id "power:GND") (at 174.625 99.06 0) (unit 1)
-    (in_bom yes) (on_board yes) (fields_autoplaced)
-    (property "Reference" "#PWR0128" (id 0) (at 174.625 105.41 0)
-      (effects (font (size 1.27 1.27)) hide)
-    )
-    (property "Value" "GND" (id 1) (at 174.625 103.505 0))
-    (property "Footprint" "" (id 2) (at 174.625 99.06 0)
-      (effects (font (size 1.27 1.27)) hide)
-    )
-    (property "Datasheet" "" (id 3) (at 174.625 99.06 0)
       (effects (font (size 1.27 1.27)) hide)
     )
@@
     (pin "2")
   )
-  (symbol (lib_id "power:GND") (at 142.875 114.3 0) (unit 1)
-    (in_bom yes) (on_board yes) (fields_autoplaced)
-    (property "Reference" "#PWR0121" (id 0) (at 142.875 120.65 0)
-      (effects (font (size 1.27 1.27)) hide)
-    )
-    (property "Value" "GND" (id 1) (at 142.875 119.38 0))
-    (property "Footprint" "" (id 2) (at 142.875 114.3 0)
-      (effects (font (size 1.27 1.27)) hide)
-    )
-    (property "Datasheet" "" (id 3) (at 142.875 114.3 0)
-      (effects (font (size 1.27 1.27)) hide)
-    )
-    (pin "1")
-  )
   (symbol (lib_id "Device:R") (at 99.695 110.49 0) (unit 1)

Commit message: finished up V1.0. Review required
Other:
- company: (none) -> HAN
- title: (none) -> Water Quality Monitor
Changed lines of the file:
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@@
 (kicad_sch (version 20211123) (generator eeschema)
   (paper "A4")
+  (title_block
+    (title "Water Quality Monitor")
+    (rev "1")
+    (company "HAN")
+    (comment 1 "Casper R. Tak")
+  )
   (junction (at 185.42 98.425) (diameter 0) (color 0 0 0 0)
   )
