File: Hardware/Rastaban-HAT/Rastaban-HAT/3.3V&5.kicad_sch (KiCad schematic)
At the start: 17 parts, among them U8 RT7272AGSP

Commit message: cleanup and changed some names to Rastaban
Other:
- title: Water Quality Monitor -> Rastaban-HAT
Changed lines of the file:
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@@
   (paper "A4")
   (title_block
-    (title "Water Quality Monitor")
+    (title "Rastaban-HAT")
     (rev "1")
     (company "HAN")
