File: Hardware/Rastaban-HAT/Rastaban-HAT/FluidMotors.kicad_sch (KiCad schematic)
At the start: 14 parts, among them U3 TMC2208_Carrier, U4 TMC2208_Carrier

Commit message: added new libarries and jlcpcb part plugin
Parts:
- C16: value 100u 35V -> 100uF 35V; footprint (none) -> Capacitor_THT:C_Radial_D6.3mm_H5.0mm_P2.50mm; Manufacturer_Part_Number (none) -> C3339
- C17: value 100u 35V -> 100uF 35V; footprint (none) -> Capacitor_THT:C_Radial_D6.3mm_H11.0mm_P2.50mm; Manufacturer_Part_Number (none) -> C3339
- C22, C23: value 100nF -> 100nF 6.3V; footprint (none) -> Capacitor_SMD:C_0805_2012Metric_Pad1.18x1.45mm_HandSolder
- JP2, JP3: footprint (none) -> Jumper:SolderJumper-3_P1.3mm_Open_Pad1.0x1.5mm_NumberLabels
- R20, R21, R22, R23: footprint Resistor_SMD:R_1206_3216Metric_Pad1.30x1.75mm_HandSolder -> Resistor_SMD:R_0805_2012Metric_Pad1.20x1.40mm_HandSolder
- U3, U4: footprint Footprints:TMC2208_SILENTSTEPSTICK -> (none)
Changed lines of the file:
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@@
     (property "Reference" "U4" (id 0) (at 184.15 78.74 0))
     (property "Value" "TMC2208_Carrier" (id 1) (at 184.15 81.28 0))
-    (property "Footprint" "Footprints:TMC2208_SILENTSTEPSTICK" (id 2) (at 168.91 123.19 0)
+    (property "Footprint" "" (id 2) (at 168.91 123.19 0)
       (effects (font (size 1.27 1.27)) (justify left bottom) hide)
     )
@@
     (property "Reference" "JP2" (id 0) (at 132.715 75.565 0))
     (property "Value" "Jumper_3_Open" (id 1) (at 132.715 78.105 0))
-    (property "Footprint" "" (id 2) (at 132.715 82.55 0)
+    (property "Footprint" "Jumper:SolderJumper-3_P1.3mm_Open_Pad1.0x1.5mm_NumberLabels" (id 2) (at 132.715 82.55 0)
       (effects (font (size 1.27 1.27)) hide)
     )
@@
       (effects (font (size 1.27 1.27)) (justify left))
     )
-    (property "Footprint" "Resistor_SMD:R_1206_3216Metric_Pad1.30x1.75mm_HandSolder" (id 2) (at 151.892 114.3 90)
+    (property "Footprint" "Resistor_SMD:R_0805_2012Metric_Pad1.20x1.40mm_HandSolder" (id 2) (at 151.892 114.3 90)
       (effects (font (size 1.27 1.27)) hide)
     )
@@
     (property "Reference" "JP3" (id 0) (at 211.455 75.565 0))
     (property "Value" "Jumper_3_Open" (id 1) (at 211.455 78.105 0))
-    (property "Footprint" "" (id 2) (at 211.455 82.55 0)
+    (property "Footprint" "Jumper:SolderJumper-3_P1.3mm_Open_Pad1.0x1.5mm_NumberLabels" (id 2) (at 211.455 82.55 0)
       (effects (font (size 1.27 1.27)) hide)
     )
@@
       (effects (font (size 1.27 1.27)) (justify left))
     )
-    (property "Value" "100nF" (id 1) (at 213.36 94.6149 0)
-      (effects (font (size 1.27 1.27)) (justify left))
-    )
-    (property "Footprint" "" (id 2) (at 211.1502 97.155 0)
+    (property "Value" "100nF 6.3V" (id 1) (at 213.36 94.6149 0)
+      (effects (font (size 1.27 1.27)) (justify left))
+    )
+    (property "Footprint" "Capacitor_SMD:C_0805_2012Metric_Pad1.18x1.45mm_HandSolder" (id 2) (at 211.1502 97.155 0)
       (effects (font (size 1.27 1.27)) hide)
     )
@@
       (effects (font (size 1.27 1.27)) (justify left))
     )
-    (property "Footprint" "Resistor_SMD:R_1206_3216Metric_Pad1.30x1.75mm_HandSolder" (id 2) (at 79.502 114.3 90)
+    (property "Footprint" "Resistor_SMD:R_0805_2012Metric_Pad1.20x1.40mm_HandSolder" (id 2) (at 79.502 114.3 90)
       (effects (font (size 1.27 1.27)) hide)
     )
@@
       (effects (font (size 1.27 1.27)) (justify left))
     )
-    (property "Footprint" "Resistor_SMD:R_1206_3216Metric_Pad1.30x1.75mm_HandSolder" (id 2) (at 158.242 114.3 90)
+    (property "Footprint" "Resistor_SMD:R_0805_2012Metric_Pad1.20x1.40mm_HandSolder" (id 2) (at 158.242 114.3 90)
       (effects (font (size 1.27 1.27)) hide)
     )
@@
       (effects (font (size 1.27 1.27)) (justify left))
     )
-    (property "Value" "100u 35V" (id 1) (at 139.7 102.2349 0)
-      (effects (font (size 1.27 1.27)) (justify left))
-    )
-    (property "Footprint" "" (id 2) (at 136.8552 104.775 0)
+    (property "Value" "100uF 35V" (id 1) (at 139.7 102.2349 0)
+      (effects (font (size 1.27 1.27)) (justify left))
+    )
+    (property "Footprint" "Capacitor_THT:C_Radial_D6.3mm_H5.0mm_P2.50mm" (id 2) (at 136.8552 104.775 0)
       (effects (font (size 1.27 1.27)) hide)
     )
     (property "Datasheet" "~" (id 3) (at 135.89 100.965 0)
+      (effects (font (size 1.27 1.27)) hide)
+    )
+    (property "LCSC Part#" "" (id 4) (at 135.89 100.965 0)
+      (effects (font (size 1.27 1.27)) hide)
+    )
+    (property "Manufacturer_Part_Number" "C3339" (id 5) (at 135.89 100.965 0)
       (effects (font (size 1.27 1.27)) hide)
     )
@@
     (property "Reference" "U3" (id 0) (at 106.045 78.74 0))
     (property "Value" "TMC2208_Carrier" (id 1) (at 106.045 81.28 0))
-    (property "Footprint" "Footprints:TMC2208_SILENTSTEPSTICK" (id 2) (at 90.805 123.19 0)
+    (property "Footprint" "" (id 2) (at 90.805 123.19 0)
       (effects (font (size 1.27 1.27)) (justify left bottom) hide)
     )
@@
       (effects (font (size 1.27 1.27)) (justify left))
     )
-    (property "Footprint" "Resistor_SMD:R_1206_3216Metric_Pad1.30x1.75mm_HandSolder" (id 2) (at 73.152 114.3 90)
+    (property "Footprint" "Resistor_SMD:R_0805_2012Metric_Pad1.20x1.40mm_HandSolder" (id 2) (at 73.152 114.3 90)
       (effects (font (size 1.27 1.27)) hide)
     )
@@
       (effects (font (size 1.27 1.27)) (justify left))
     )
-    (property "Value" "100u 35V" (id 1) (at 219.71 102.2349 0)
-      (effects (font (size 1.27 1.27)) (justify left))
-    )
-    (property "Footprint" "" (id 2) (at 217.5002 104.775 0)
+    (property "Value" "100uF 35V" (id 1) (at 219.71 102.2349 0)
+      (effects (font (size 1.27 1.27)) (justify left))
+    )
+    (property "Footprint" "Capacitor_THT:C_Radial_D6.3mm_H11.0mm_P2.50mm" (id 2) (at 217.5002 104.775 0)
       (effects (font (size 1.27 1.27)) hide)
     )
     (property "Datasheet" "~" (id 3) (at 216.535 100.965 0)
+      (effects (font (size 1.27 1.27)) hide)
+    )
+    (property "LCSC Part#" "" (id 4) (at 216.535 100.965 0)
+      (effects (font (size 1.27 1.27)) hide)
+    )
+    (property "Manufacturer_Part_Number" "C3339" (id 5) (at 216.535 100.965 0)
       (effects (font (size 1.27 1.27)) hide)
     )
@@
       (effects (font (size 1.27 1.27)) (justify left))
     )
-    (property "Value" "100nF" (id 1) (at 135.89 94.6149 0)
-      (effects (font (size 1.27 1.27)) (justify left))
-    )
-    (property "Footprint" "" (id 2) (at 133.0452 97.155 0)
-      (effects (font (size 1.27 1.27)) hide)
-    )
+    (property "Value" "100nF 6.3V" (id 1) (at 135.89 94.6149 0)
+      (effects (font (size 1.27 1.27)) (justify left))
+    )
+    (property "Footprint" "Capacitor_SMD:C_0805_2012Metric_Pad1.18x1.45mm_HandSolder" (id 2) (at 133.0452 97.155 0)
+      (effects (font (size 1.27 1.27)) hide)
+    )

Commit message: updated footprints
Parts:
- U3, U4: footprint (none) -> SnapEDA Library:MODULE_TMC2208_SILENTSTEPSTICK
Changed lines of the file:
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@@
     (property "Reference" "U4" (id 0) (at 184.15 78.74 0))
     (property "Value" "TMC2208_Carrier" (id 1) (at 184.15 81.28 0))
-    (property "Footprint" "" (id 2) (at 168.91 123.19 0)
+    (property "Footprint" "SnapEDA Library:MODULE_TMC2208_SILENTSTEPSTICK" (id 2) (at 168.91 123.19 0)
       (effects (font (size 1.27 1.27)) (justify left bottom) hide)
     )
@@
     (property "Reference" "U3" (id 0) (at 106.045 78.74 0))
     (property "Value" "TMC2208_Carrier" (id 1) (at 106.045 81.28 0))
-    (property "Footprint" "" (id 2) (at 90.805 123.19 0)
+    (property "Footprint" "SnapEDA Library:MODULE_TMC2208_SILENTSTEPSTICK" (id 2) (at 90.805 123.19 0)
       (effects (font (size 1.27 1.27)) (justify left bottom) hide)
     )

Commit message: ERC fixed on schematic
Changed lines of the file:
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@@
     (comment 1 "Casper R. Tak")
   )
+  (junction (at 216.535 86.36) (diameter 0) (color 0 0 0 0)
+  )
   (junction (at 201.93 95.25) (diameter 0) (color 0 0 0 0)
   )
   (junction (at 201.93 91.44) (diameter 0) (color 0 0 0 0)
+  )
+  (junction (at 135.89 86.36) (diameter 0) (color 0 0 0 0)
   )
   (junction (at 157.48 118.11) (diameter 0) (color 0 0 0 0)
@@
     (pin "2")
   )
+  (symbol (lib_id "power:PWR_FLAG") (at 135.89 86.36 270) (unit 1)
+    (in_bom yes) (on_board yes) (fields_autoplaced)
+    (property "Reference" "#FLG0105" (id 0) (at 137.795 86.36 0)
+      (effects (font (size 1.27 1.27)) hide)
+    )
+    (property "Value" "PWR_FLAG" (id 1) (at 139.7 86.3599 90)
+      (effects (font (size 1.27 1.27)) (justify left))
+    )
+    (property "Footprint" "" (id 2) (at 135.89 86.36 0)
+      (effects (font (size 1.27 1.27)) hide)
+    )
+    (property "Datasheet" "~" (id 3) (at 135.89 86.36 0)
+      (effects (font (size 1.27 1.27)) hide)
+    )
+    (pin "1")
+  )
+  (symbol (lib_id "power:PWR_FLAG") (at 216.535 86.36 270) (unit 1)
+    (in_bom yes) (on_board yes) (fields_autoplaced)
+    (property "Reference" "#FLG0103" (id 0) (at 218.44 86.36 0)
+      (effects (font (size 1.27 1.27)) hide)
+    )
+    (property "Value" "PWR_FLAG" (id 1) (at 220.345 86.3599 90)
+      (effects (font (size 1.27 1.27)) (justify left))
+    )
+    (property "Footprint" "" (id 2) (at 216.535 86.36 0)
+      (effects (font (size 1.27 1.27)) hide)
+    )
+    (property "Datasheet" "~" (id 3) (at 216.535 86.36 0)
+      (effects (font (size 1.27 1.27)) hide)
+    )
+    (pin "1")
+  )
   (symbol (lib_id "power:GND") (at 203.2 118.11 0) (unit 1)

Commit message: removed warnings in PCB new by fixing footprints
Parts:
- removed U4: TMC2208_Carrier, SnapEDA Library:MODULE_TMC2208_SILENTSTEPSTICK, symbol TMC2208_SILENTSTEPSTICK:TMC2208_SILENTSTEPSTICK
- added U?: TMC2208_Carrier, SnapEDA Library:MODULE_TMC2208_SILENTSTEPSTICK, symbol TMC2208_SILENTSTEPSTICK:TMC2208_SILENTSTEPSTICK
- TP3, TP4: footprint TestPoint:TestPoint_Bridge_Pitch7.62mm_Drill1.3mm -> TestPoint:TestPoint_THTPad_2.0x2.0mm_Drill1.0mm
Connections:
- net 3.3V+: now also U?.JP2_7 (VIO); no longer C23.2
- net DIRSEC: now also U?.JP1_1 (DIR)
- net ENSEC: now also U?.JP1_8 (EN)
- net GND: now also U?.JP2_2 (GND), U?.JP2_8 (GND)
- net OA1SEC: now also U?.JP2_4 (OA1)
- net OA2SEC: now also U?.JP2_3 (OA2)
- net OB1SEC: now also U?.JP2_5 (OB1)
- net OB2SEC: now also U?.JP2_6 (OB2)
- net STEPSEC: now also U?.JP1_2 (STEP)
- net at R23.1: now also U?.JP1_6 (MS2)
- net at R22.1: now also U?.JP1_7 (MS1)
- net at C17.1, JP3.2 (C): now also U?.JP2_1 (VM)
- net DIAGPRI: no longer names the net of U3.JP3_1 (DIAG)
- new net: C23.2, U?.VREF
- no-connect marks 6 -> 10

Commit message: finished drv8838 implementation for PCBNEW
Parts:
- gave numbers to parts that had none: 1
Changed lines of the file:
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@@
   (symbol (lib_name "TMC2208_SILENTSTEPSTICK_1") (lib_id "TMC2208_SILENTSTEPSTICK:TMC2208_SILENTSTEPSTICK") (at 184.15 104.14 0) (unit 1)
     (in_bom yes) (on_board yes)
-    (property "Reference" "U?" (id 0) (at 184.15 78.74 0))
+    (property "Reference" "U4" (id 0) (at 184.15 78.74 0))
     (property "Value" "TMC2208_Carrier" (id 1) (at 184.15 81.28 0))
     (property "Footprint" "SnapEDA Library:MODULE_TMC2208_SILENTSTEPSTICK" (id 2) (at 168.91 123.19 0)
