File: Hardware/Rastaban-HAT/Workmap Rastaban-HAT/Rastaban-HAT.kicad_sch (KiCad schematic)
At the start: 55 parts, among them J1 1778780, J10 GPIO, J11 Conn_01x06_Male, J2 1778780, J3 1778780, J4 Screw_Terminal_01x02, J5 Jack-DC 12V+, J6 SM04B-SRSS-TB(LF)(SN), J7 Screw_Terminal_01x02, J8 Screw_Terminal_01x02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

Commit message: testscript made
Parts:
- PE1: Purpose (none) -> 12V peltier module for heating and cooling
Changed lines of the file:
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@@
+      (effects (font (size 1.27 1.27)) hide)
+    )
+    (property "Purpose" "12V peltier module for heating and cooling" (id 6) (at 60.325 127.635 0)
       (effects (font (size 1.27 1.27)) hide)
     )
